Commit message: WIP snapshot: HG-DAgger architecture, joystick/pause-resume, gripper-capture fix, session docs
Preserves all in-progress work from this session before a stop:
- ffw_joystick_controller pause/resume + home-pose idle-publish suppression
- config/urdf/xacro changes for the a2 leader + sg2 follower
- tmp_readmes/: HG-DAgger architecture diagram (tex+pdf), session memory, and related docs

See tmp_readmes/SESSION_MEMORY.md for full context and how to port this back.

Co-Authored-By: Claude Sonnet 5 <noreply@anthropic.com>

File: ffw_description/ros2_control/ffw_a2_leader/ffw_a2_leader.ros2_control.xacro (robot description, xacro)
@@ -18,5 +18,5 @@
           <xacro:unless value="${use_mock_hardware}">
             <plugin>dynamixel_hardware_interface/DynamixelHardware</plugin>
-            <param name="port_name">/dev/serial/by-role/leader_a2</param>
+            <param name="port_name">/dev/serial/by-id/usb-ROBOTIS_Avatar_Controller_357A396C3235-if00</param>
             <param name="baud_rate">4000000</param>
             <param name="dynamixel_model_folder">/param/dxl_model</param>

File: ffw_description/urdf/common/follower/ffw_follower_body.xacro (robot description, xacro)
@@ -42,5 +42,8 @@
          <origin xyz="0.049483 0 0.102130" rpy="0 0 0" />
          <axis xyz="0 1 0" />
-         <limit velocity="4.8" effort="1000" lower="-0.2317" upper="0.6951" />
+         <!-- Upper limit raised from 0.6951 to 0.90. Teleop recordings reach a
+              head pitch of ~0.862 (Task_150_2bottlespplf), so the old bound sat
+              below the mechanical range and clipped the AI task camera view. -->
+         <limit velocity="4.8" effort="1000" lower="-0.2317" upper="0.90" />
          <dynamics damping="0.1" />
       </joint>

File: ffw_description/urdf/ffw_sg2_rev1_follower/ffw_sg2_follower.urdf (robot description, URDF)
Before this commit: robot ffw_sg2_follower, 50 links, 49 joints
Joints:
- joint head_joint1: limit lower=-0.2317 upper=0.6951 effort=1000 velocity=4.8 -> lower=-0.2317 upper=0.90 effort=1000 velocity=4.8
